File: hardware/pro/propmesh/motors.kicad_sch (KiCad schematic)
At the start: 32 parts, among them J15 MS_SEL, J16 DIAG_AUX, J19 MS_SEL, J20 MS_SEL, J21 MS_SEL, J22 MS_SEL, J23 MS_SEL, J24 DIAG_AUX, Q8 AO3400A

Commit message: Sheet 07 (sensors + expansion) captured; sheet 05 spec ready
Sheet 07 drawn and verified: 3 clamped digital inputs (+ PIR header),
2 halved analog inputs, TSOP38238 on filtered 3V3, Qwiic (SH-1.0 clone
C7430446 — genuine JST stock-dead), 2x5 expansion header with GPIO45/46
strap protection. checknet all green, ERC clean bar the 4 LED labels
awaiting sheet 05. D2_MID global on motors + sensors sheets so
expansion pin 9 rides GPIO43's 1k.

Sheet 05 spec: AHCT125 moved to SOIC-14 C155176 (TSSOP dead at JLC),
strip 2 = 2x DG128-02P (04P dead), WS2812B-MINI-X2 status pixel
imported + datasheet-verified (pins, land pattern, VIH math).

Cost: all seven blocks now verified; parts subtotal $31.93,
duty-paid ~$48.55. Open item #2 mostly resolved (residual: JLC order
UI check before first PCBA run).

New repo rule after the C_A1 collision: spec refs are project-global —
never reuse one across sheet yamls (audio R_D3 -> R_DAT3, sensor caps
-> C_AN1/2).

Co-Authored-By: Claude Fable 5 <noreply@anthropic.com>
Changed lines of the file:
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@@
-		)
-	)
-	(label "D2_MID"
-		(at 45.72 95.25 0)
-		(effects
-			(font
-				(size 1.27 1.27)
-			)
-			(justify left bottom)
 		)
 	)
@@
 			(hide yes)
 			(show_name no)
+			(do_not_autoplace no)
+			(effects
+				(font
+					(size 1.27 1.27)
+				)
+				(justify left)
+			)
+		)
+	)
+	(global_label "D2_MID"
+		(shape input)
+		(at 49.53 95.25 90)
+		(fields_autoplaced yes)
+		(effects
+			(font
+				(size 1.27 1.27)
+			)
+			(justify left)
+		)
+		(property "Intersheetrefs" "${INTERSHEET_REFS}"
+			(at 49.53 85.4915 90)
+			(hide yes)
+			(show_name no)

Commit message: Pro schematic complete; enclosure, layout guide, timeline and radio decisions
Schematic: all seven design sheets drawn and green; project-wide ERC at
zero. IR receiver dropped (hidden board can't see a remote — plug-in on
a DIGITAL_IN); GPIO 3 became LED_STRIP_1_CLK; both strip outputs 3- or
4-wire through one octal SN74AHCT541DWR (three revisions of the shifter
in one day, no mode jumpers). Input FET symbol replaced: KiCad 10's
Device:Q_PMOS numbers pins D/G/S and matches no pad — the part would
have been unconnected with no ERC/DRC complaint. All 196 references
renumbered to standard sequential designators (yaml keeps spec names;
the checker prints both). Sheet 08 (test points) and the sheet 01
staged-power link headers specified per spec §2.6 — sheet 01's checker
is red until they are drawn.

checknet.py: symbol pins ⊆ footprint pads check (the silent killer),
multi-unit pin keys + per-unit diagrams (`units:`), symbol-vote sheet
anchoring for half-drawn sheets, orientation-aware net voting, foreign
part reporting, cross-sheet extras no longer crash the report.

Docs: hardware/pro/layout.md — placement by designator, IPC-2221 trace
widths, thermal, silk, ⚠ list, KiCad primer; every chip's datasheet
layout section read (WROOM-1U has NO keep-out; DRV8871 wants a bottom
GND pour; MAX98357A output-trace numbers). Enclosure plan (spec §2.3):
Multilink RNI-1500 / RNI-300, DRiBOX Medium, Joinfworld clear-lid box,
icotek KEL-DPZ entry plate, fit rule 210×140×60 mm inside; PSU
defaults (§2.9) and the 10 A input-path note. Software plan: timeline
design (ramps native, live scrub v1, Cue.start_offset_ms in schema),
yard access (walk-up AP, WireGuard-in-firmware, BYO remote), WiFi-PHY
radio decision vs Zigbee/BLE/LoRa, console served-from-bridge budget,
USB stays in CDC/JTAG mode (no auto-program transistors needed).

Co-Authored-By: Claude Fable 5.1 <noreply@anthropic.com>
Parts:
- renumbered C_BS1 to C18, C_BS2 to C19, C_MA1 to C20, C_MA2 to C21, C_MB1 to C22, C_MB2 to C23, J_S1L1 to J19, J_S1R1 to J20, J16 to J21, J_S2R1 to J22, J_MA1 to J23, J_S2L1 to J24, XH1 to J25, J24 to J26, XH2 to J27, J_MB1 to J28, J21 to J29, J15 to J30, J22 to J31, J19 to J32, J23 to J33, J20 to J34, JP3 to JP2, R31 to R22, R29 to R23, R30 to R24, R_UTX1 to R25, R_ENP1 to R26, U_MA1 to U7, U_MB1 to U8

Commit message: Pro v0.1: board setup + placement, two design reviews applied, datasheet-review changes specced
Checkpoint of two weeks' work since dacce25. The schematic is MID-EDIT:
sheets 02/04/05/07/08 checkers are red by design until the changes in
hardware/pro/schematic-changes-2026-09-16.md are drawn; sheet 03 is
half-drawn (see finish-v0.1.md).

Layout
- layout.md rebuilt as one ordered procedure (Part A) with a
  where-you-are line; Board Setup, outline, origin, frozen 120x90 hole
  pattern; routing and pour guidance; per-net noise keep-outs
- tools: checksetup.py (setup/outline/holes/netclasses/socket rows),
  placeboard.py, placetps.py (test points on B.Cu for bodge + pogo rig),
  setpos.py, snapgrid.py; placement renders; power/MCU placement tables

Reviews
- review-2026-09-08 (external audit): C1 EN cap, MA/MB_ILIM short,
  servo/output channel order, sensor clamp order, VIN_FUSED label,
  F1 footprint — all fixed in the schematic
- checknet.py: merged-net assertion (distinct spec nets must be
  distinct schematic nets) — the class that hid the ILIM short
- review-2026-09-16 (routing) + datasheet-review-2026-09-16 with a
  verified disposition; Mini plan audit + recommendations (other session)

Decisions 2026-09-16 (specs, pinmap and headers updated; drawing pending)
- 5 V rail: strip bulk 1000 uF -> 220 uF Rubycon C88757; JP_USB link
  makes USB power opt-in (AP64350 hiccups into 2 mF)
- sensor series R 1 k 0603 -> 2.2 k 1206 C17948 (24 V miswire)
- second PCA9685 (0x41, 1 kHz) for the six DC channels; servos stay at
  50 Hz on 0x40; both OE on GPIO 37 = PCA_OE with pull-up (pinmap:
  36/36 GPIO used; genpins.py supports several PCA9685s)
- output FETs Q1-Q6 -> 40 V Vishay SI2356DS C74127 (TVS coordination)
- SD DAT1/DAT2 pull-ups; USB 22R pair + DNP caps + VBUS 100 nF;
  74AHCT541 input pulldowns, R53 fitted
- MP6603 dual-mode socket mapping verified; MS strap defaults decided

Co-Authored-By: Claude Opus 5 (1M context) <noreply@anthropic.com>
Connections:
- net MA_ILIM: no longer R24.1, U8.4 (ILIM)
- new net MB_ILIM: R24.1, U8.4 (ILIM)
Changed lines of the file:
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@@
 		)
 	)
-	(label "MA_ILIM"
+	(label "MB_ILIM"
 		(at 182.88 102.87 0)
 		(effects
@@
 		(dnp no)
 		(property "Reference" "J28"
-			(at 263.906 92.964 0)
+			(at 263.906 92.964 90)
 			(show_name no)
 			(do_not_autoplace no)
