File: hardware/pro/propmesh/leds.kicad_sch (KiCad schematic)
At the start: 0 parts

Commit message: Pro schematic complete; enclosure, layout guide, timeline and radio decisions
Schematic: all seven design sheets drawn and green; project-wide ERC at
zero. IR receiver dropped (hidden board can't see a remote — plug-in on
a DIGITAL_IN); GPIO 3 became LED_STRIP_1_CLK; both strip outputs 3- or
4-wire through one octal SN74AHCT541DWR (three revisions of the shifter
in one day, no mode jumpers). Input FET symbol replaced: KiCad 10's
Device:Q_PMOS numbers pins D/G/S and matches no pad — the part would
have been unconnected with no ERC/DRC complaint. All 196 references
renumbered to standard sequential designators (yaml keeps spec names;
the checker prints both). Sheet 08 (test points) and the sheet 01
staged-power link headers specified per spec §2.6 — sheet 01's checker
is red until they are drawn.

checknet.py: symbol pins ⊆ footprint pads check (the silent killer),
multi-unit pin keys + per-unit diagrams (`units:`), symbol-vote sheet
anchoring for half-drawn sheets, orientation-aware net voting, foreign
part reporting, cross-sheet extras no longer crash the report.

Docs: hardware/pro/layout.md — placement by designator, IPC-2221 trace
widths, thermal, silk, ⚠ list, KiCad primer; every chip's datasheet
layout section read (WROOM-1U has NO keep-out; DRV8871 wants a bottom
GND pour; MAX98357A output-trace numbers). Enclosure plan (spec §2.3):
Multilink RNI-1500 / RNI-300, DRiBOX Medium, Joinfworld clear-lid box,
icotek KEL-DPZ entry plate, fit rule 210×140×60 mm inside; PSU
defaults (§2.9) and the 10 A input-path note. Software plan: timeline
design (ramps native, live scrub v1, Cue.start_offset_ms in schema),
yard access (walk-up AP, WireGuard-in-firmware, BYO remote), WiFi-PHY
radio decision vs Zigbee/BLE/LoRa, console served-from-bridge budget,
USB stays in CDC/JTAG mode (no auto-program transistors needed).

Co-Authored-By: Claude Fable 5.1 <noreply@anthropic.com>
Parts:
- added C42, C44: 100n, Capacitor_SMD:C_0603_1608Metric, symbol Device:C
- added C43, C45: 1000u/16V, Capacitor_THT:CP_Radial_D10.0mm_P5.00mm, symbol Device:C_Polarized
- added J36: LED2_SIG, propmesh:CONN-TH_DG128-5.0-02P-14-00A-H, symbol Connector:Screw_Terminal_01x02
- added J37: LED1_SIG, propmesh:CONN-TH_DG128-5.0-02P-14-00A-H, symbol Connector:Screw_Terminal_01x02
- added J38: LED1_PWR, propmesh:CONN-TH_DG128-5.0-02P-14-00A-H, symbol Connector:Screw_Terminal_01x02
- added J39: LED2_PWR, propmesh:CONN-TH_DG128-5.0-02P-14-00A-H, symbol Connector:Screw_Terminal_01x02
- added LED1: WS2812B-MINI, propmesh:LED-SMD_4P-L3.5-W3.5-TL_WS2812B-1, symbol propmesh:WS2812B-MINI-X1
- added R34, R35, R36, R37, R38: 330R, Resistor_SMD:R_0603_1608Metric, symbol Device:R
- added U11: SN74AHCT541, Package_SO:SOIC-20W_7.5x12.8mm_P1.27mm, symbol 74xx:74AHCT541
Connections:
- new net: R34.1, U11.17 (Y1)
- new net: J37.2 (Pin_2), R34.2
- new net: R38.2, U11.14 (Y4)
- new net: R37.1, U11.15 (Y3)
- new net: R36.1, U11.16 (Y2)
- new net: R35.1, U11.18 (Y0)
- new net: LED1.1 (DIN), R38.1
- new net: J36.2 (Pin_2), R37.2
- new net: J37.1 (Pin_1), R35.2
- new net: J36.1 (Pin_1), R36.2
- new net +5V: C42.1, C43.1, C44.1, C45.1, J38.1 (Pin_1), J39.1 (Pin_1), LED1.2 (VDD), U11.20 (VCC)
- new net GND: C42.2, C43.2, C44.2, C45.2, J38.2 (Pin_2), J39.2 (Pin_2), LED1.4 (GND), U11.1 (G1), U11.10 (GND), U11.19 (G2), U11.7 (A5), U11.8 (A6), U11.9 (A7)
- new net LED_STRIP_1_CLK: U11.3 (A1)
- new net LED_STRIP_1_DATA: U11.2 (A0)
- new net LED_STRIP_2_CLK: U11.5 (A3)
- new net LED_STRIP_2_DATA: U11.4 (A2)
- new net STATUS_LED: U11.6 (A4)
- no-connect marks 0 -> 4

Commit message: Pro v0.1 schematic complete; board cleanup pass, parity 0
Schematic: all datasheet-review changes drawn (decisions 1A, 2A, 3B,
OE on GPIO 37, 4B). All eight sheet checkers ALL NETS MATCH, ERC 0
errors / 0 warnings, pinmap matches generated headers.
- sheet 03: second PCA9685 (U12, 0x41) with B-straps, PCA_OE net with
  10k pull-up (R59); DC FETs Q1-Q6 = SI2356DS
- sheets 02/04/05/07/08: USB link/22R/VBUS cap, SD DAT1/DAT2 pull-ups,
  shifter pulldowns, 2.2k 1206 sensor Rs; R53 (GPIO3 pulldown) now drawn
  on sheet 05, specs moved to match

Board (KiCad closed, backup kept):
- F8 done, schematic parity 0; orphan DNP R53 removed
- mounting holes H1-H4, board-only, excluded from BOM/position files
- minimum drill 0.3 -> 0.2 mm: U2's own 0.2/0.6 thermal vias; JLCPCB
  4-layer standard cost for 0.2 mm holes with >= 0.45 mm pads
- DG128-02P pads 2.3 -> 2.8 mm (J17 10 A input; library edited too)
- DRV8871 exposed-pad paste inset 0.1 mm (library edited too)
- 43 parts snapped to grid; snapgrid.py now exempts J20/J22 so the
  StepStick rows stay 12.70 mm
- DRC: 11 courtyard overlaps left (3 accepted terminal gangs, 8 in the
  sensor corner from the 1206 resistors) + silkscreen

Tools: checknet.py net vote ignores orientation for R/C/L (three
upside-down pull-ups had out-voted the chip pin on sheet 04); verified
it still catches a shorted net and a mis-wired pull-up.
checksetup.py: min drill 0.2.

Also includes the Mini module selection and KiCad project started in
another session (2026-09-19).

Co-Authored-By: Claude Opus 5.5 <noreply@anthropic.com>
Parts:
- added R53: 10k, Resistor_SMD:R_0603_1608Metric, symbol Device:R
- added R61, R62, R63, R64: 10K, Resistor_SMD:R_0603_1608Metric, symbol Device:R
- C43, C45: value 1000u/16V -> 220u/16V; footprint Capacitor_THT:CP_Radial_D10.0mm_P5.00mm -> Capacitor_THT:CP_Radial_D6.3mm_P2.50mm
Connections:
- net GND: now also R53.2, R61.2, R62.2, R63.2, R64.2
- net LED_STRIP_1_CLK: now also R53.1
- net LED_STRIP_1_DATA: now also R61.1
- net LED_STRIP_2_CLK: now also R63.1
- net LED_STRIP_2_DATA: now also R62.1
- net STATUS_LED: now also R64.1
Other:
- moved on the sheet: C42, C43, C44, C45, J36, J37, J38, J39, LED1, R34, R35, R36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
