File: hardware/pro/propmesh/outputs.kicad_sch (KiCad schematic)
At the start: 42 parts, among them J10 SERVO, J11 SERVO, J12 SERVO, J13 SERVO, J3 RELAY_OUT, J6 RELAY_OUT, J7 SERVO, J8 RELAY_OUT, J9 SERVO, K1 HK4100F-DC5V-SHG, K2 HK4100F-DC5V-SHG, K3 HK4100F-DC5V-SHG, Q1 AO3400A, Q3 AO3400A, Q4 AO3400A, Q5 AO3400A, Q6 AO3400A, Q7 AO3400A, U5 PCA9685PW, U6 ULN2003A

Commit message: Pro schematic complete; enclosure, layout guide, timeline and radio decisions
Schematic: all seven design sheets drawn and green; project-wide ERC at
zero. IR receiver dropped (hidden board can't see a remote — plug-in on
a DIGITAL_IN); GPIO 3 became LED_STRIP_1_CLK; both strip outputs 3- or
4-wire through one octal SN74AHCT541DWR (three revisions of the shifter
in one day, no mode jumpers). Input FET symbol replaced: KiCad 10's
Device:Q_PMOS numbers pins D/G/S and matches no pad — the part would
have been unconnected with no ERC/DRC complaint. All 196 references
renumbered to standard sequential designators (yaml keeps spec names;
the checker prints both). Sheet 08 (test points) and the sheet 01
staged-power link headers specified per spec §2.6 — sheet 01's checker
is red until they are drawn.

checknet.py: symbol pins ⊆ footprint pads check (the silent killer),
multi-unit pin keys + per-unit diagrams (`units:`), symbol-vote sheet
anchoring for half-drawn sheets, orientation-aware net voting, foreign
part reporting, cross-sheet extras no longer crash the report.

Docs: hardware/pro/layout.md — placement by designator, IPC-2221 trace
widths, thermal, silk, ⚠ list, KiCad primer; every chip's datasheet
layout section read (WROOM-1U has NO keep-out; DRV8871 wants a bottom
GND pour; MAX98357A output-trace numbers). Enclosure plan (spec §2.3):
Multilink RNI-1500 / RNI-300, DRiBOX Medium, Joinfworld clear-lid box,
icotek KEL-DPZ entry plate, fit rule 210×140×60 mm inside; PSU
defaults (§2.9) and the 10 A input-path note. Software plan: timeline
design (ramps native, live scrub v1, Cue.start_offset_ms in schema),
yard access (walk-up AP, WireGuard-in-firmware, BYO remote), WiFi-PHY
radio decision vs Zigbee/BLE/LoRa, console served-from-bridge budget,
USB stays in CDC/JTAG mode (no auto-program transistors needed).

Co-Authored-By: Claude Fable 5.1 <noreply@anthropic.com>
Parts:
- renumbered C16 to C4, C17 to C5, D6 to D2, D7 to D3, D8 to D4, D9 to D5, D10 to D6, D11 to D7, J_LED2 to J10, J_LED4 to J11, J_LED5 to J12, J_LED6 to J13, J3 to J14, J6 to J15, J8 to J16, J7 to J2, J9 to J3, J10 to J4, J11 to J5, J13 to J6, J12 to J7, J_LED1 to J8, J_LED3 to J9, Q3 to Q2, Q4 to Q3, Q5 to Q4, Q6 to Q5, Q7 to Q6, R17 to R10, R18 to R11, R19 to R12, R20 to R5, R21 to R6, R14 to R7, R15 to R8, R16 to R9, U6 to U3, U5 to U4

Commit message: Pro v0.1: board setup + placement, two design reviews applied, datasheet-review changes specced
Checkpoint of two weeks' work since dacce25. The schematic is MID-EDIT:
sheets 02/04/05/07/08 checkers are red by design until the changes in
hardware/pro/schematic-changes-2026-09-16.md are drawn; sheet 03 is
half-drawn (see finish-v0.1.md).

Layout
- layout.md rebuilt as one ordered procedure (Part A) with a
  where-you-are line; Board Setup, outline, origin, frozen 120x90 hole
  pattern; routing and pour guidance; per-net noise keep-outs
- tools: checksetup.py (setup/outline/holes/netclasses/socket rows),
  placeboard.py, placetps.py (test points on B.Cu for bodge + pogo rig),
  setpos.py, snapgrid.py; placement renders; power/MCU placement tables

Reviews
- review-2026-09-08 (external audit): C1 EN cap, MA/MB_ILIM short,
  servo/output channel order, sensor clamp order, VIN_FUSED label,
  F1 footprint — all fixed in the schematic
- checknet.py: merged-net assertion (distinct spec nets must be
  distinct schematic nets) — the class that hid the ILIM short
- review-2026-09-16 (routing) + datasheet-review-2026-09-16 with a
  verified disposition; Mini plan audit + recommendations (other session)

Decisions 2026-09-16 (specs, pinmap and headers updated; drawing pending)
- 5 V rail: strip bulk 1000 uF -> 220 uF Rubycon C88757; JP_USB link
  makes USB power opt-in (AP64350 hiccups into 2 mF)
- sensor series R 1 k 0603 -> 2.2 k 1206 C17948 (24 V miswire)
- second PCA9685 (0x41, 1 kHz) for the six DC channels; servos stay at
  50 Hz on 0x40; both OE on GPIO 37 = PCA_OE with pull-up (pinmap:
  36/36 GPIO used; genpins.py supports several PCA9685s)
- output FETs Q1-Q6 -> 40 V Vishay SI2356DS C74127 (TVS coordination)
- SD DAT1/DAT2 pull-ups; USB 22R pair + DNP caps + VBUS 100 nF;
  74AHCT541 input pulldowns, R53 fitted
- MP6603 dual-mode socket mapping verified; MS strap defaults decided

Co-Authored-By: Claude Opus 5 (1M context) <noreply@anthropic.com>
Parts:
- added C48: 10U, Capacitor_SMD:C_0805_2012Metric, symbol Device:C
- added C49: 100n, Capacitor_SMD:C_0603_1608Metric, symbol Device:C
- added R54, R55, R56, R57, R58, R60: 10k, Resistor_SMD:R_0603_1608Metric, symbol Device:R
- added R59, R61: 4.7k, Resistor_SMD:R_0603_1608Metric, symbol Device:R
- added U12: PCA9685PW, Package_SO:TSSOP-28_4.4x9.7mm_P0.65mm, symbol Driver_LED:PCA9685PW
- Q1, Q2, Q3, Q4, Q5, Q6: value AO3400A -> SI2356DS
- renumbered J9 to J10, J7 to J6, J6 to J7, J10 to J9
Connections:
- net +3V3: now also C48.1, C49.1, R54.1, R59.1, R61.1, U12.28 (VDD)
- net GND: now also C48.2, C49.2, R55.2, R56.2, R57.2, R58.2, R60.2, U12.14 (VSS), U12.23 (~{OE}), U12.25 (EXTCLK)
- net I2C_SCL: now also R61.2, U12.26 (SCL)
- net I2C_SDA: now also R59.2, U12.27 (SDA)
- net LED_1: now also U12.6 (LED0); no longer U4.12 (LED6)
- net LED_2: now also U12.7 (LED1); no longer U4.13 (LED7)
- net LED_3: now also U12.8 (LED2); no longer U4.15 (LED8)
- net LED_4: now also U12.9 (LED3); no longer U4.16 (LED9)
- net LED_5: now also U12.10 (LED4); no longer U4.17 (LED10)
- net LED_6: now also U12.11 (LED5); no longer U4.18 (LED11)
- net STEPPER_EN_RAW: now also U12.22 (LED15)
- new net: R54.2, U12.1 (A0)
- new net: R55.1, U12.2 (A1)
- new net: R60.1, U12.24 (A5)
- new net: R56.1, U12.3 (A2)
- new net: R57.1, U12.4 (A3)
- new net: R58.1, U12.5 (A4)
- no-connect marks 8 -> 23
Other:
- moved on the sheet: C4, C5, D2, D3, D4, D5, D6, D7, Q1, Q2, Q3, Q4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

Commit message: Pro v0.1 schematic complete; board cleanup pass, parity 0
Schematic: all datasheet-review changes drawn (decisions 1A, 2A, 3B,
OE on GPIO 37, 4B). All eight sheet checkers ALL NETS MATCH, ERC 0
errors / 0 warnings, pinmap matches generated headers.
- sheet 03: second PCA9685 (U12, 0x41) with B-straps, PCA_OE net with
  10k pull-up (R59); DC FETs Q1-Q6 = SI2356DS
- sheets 02/04/05/07/08: USB link/22R/VBUS cap, SD DAT1/DAT2 pull-ups,
  shifter pulldowns, 2.2k 1206 sensor Rs; R53 (GPIO3 pulldown) now drawn
  on sheet 05, specs moved to match

Board (KiCad closed, backup kept):
- F8 done, schematic parity 0; orphan DNP R53 removed
- mounting holes H1-H4, board-only, excluded from BOM/position files
- minimum drill 0.3 -> 0.2 mm: U2's own 0.2/0.6 thermal vias; JLCPCB
  4-layer standard cost for 0.2 mm holes with >= 0.45 mm pads
- DG128-02P pads 2.3 -> 2.8 mm (J17 10 A input; library edited too)
- DRV8871 exposed-pad paste inset 0.1 mm (library edited too)
- 43 parts snapped to grid; snapgrid.py now exempts J20/J22 so the
  StepStick rows stay 12.70 mm
- DRC: 11 courtyard overlaps left (3 accepted terminal gangs, 8 in the
  sensor corner from the 1206 resistors) + silkscreen

Tools: checknet.py net vote ignores orientation for R/C/L (three
upside-down pull-ups had out-voted the chip pin on sheet 04); verified
it still catches a shorted net and a mis-wired pull-up.
checksetup.py: min drill 0.2.

Also includes the Mini module selection and KiCad project started in
another session (2026-09-19).

Co-Authored-By: Claude Opus 5.5 <noreply@anthropic.com>
Parts:
- removed R61: 4.7k, Resistor_SMD:R_0603_1608Metric, symbol Device:R
- R59: value 4.7k -> 10k
Connections:
- net GND: no longer U12.23 (~{OE}), U4.23 (~{OE})
- net I2C_SDA: no longer R59.2
- net STEPPER_EN_RAW: no longer U12.22 (LED15)
- net B0_STRAP: now reaches R54.2, U12.1 (A0)
- net B1_STRAP: now reaches R55.1, U12.2 (A1)
- net B5_STRAP: now reaches R60.1, U12.24 (A5)
- net B2_STRAP: now reaches R56.1, U12.3 (A2)
- net B3_STRAP: now reaches R57.1, U12.4 (A3)
- net B4_STRAP: now reaches R58.1, U12.5 (A4)
- new net PCA_OE: R59.2, U12.23 (~{OE}), U4.23 (~{OE})
- no-connect marks 23 -> 24
Other:
- moved on the sheet: R5
