File: hardware/pro/propmesh/propmesh.kicad_pcb (KiCad board)
At the start: 2 copper layers, 130 x 100 mm, 239 parts, among them CN1 LINE_OUT, J1 TYPE-C-31-M-12, J10 LED_OUT, J11 LED_OUT, J12 LED_OUT, J13 LED_OUT, J14 RELAY_OUT, J15 RELAY_OUT, J16 RELAY_OUT, J17 DC_IN, J18 DC_JACK, J19 SOCKET_1x8, J2 SERVO, J20 SOCKET_1x8, J21 DIAG_AUX, J22 SOCKET_1x8, J23 MOTOR_OUT, J24 SOCKET_1x8, J25 STEPPER_COIL, J26 DIAG_AUX, J27 STEPPER_COIL, J28 MOTOR_OUT, J29 MS_SEL, J3 SERVO, J30 MS_SEL, J31 MS_SEL, J32 MS_SEL, J33 MS_SEL, J34 MS_SEL, J35 SPEAKER, J36 LED2_SIG, J37 LED1_SIG, J38 LED1_PWR, J39 LED2_PWR, J4 SERVO, J40 ANA_IN, J41 DIG_IN, J42 EXPANSION, J43 ANA_IN, J44 DIG_IN, J45 DIG_IN, J46 PIR_HDR, J47 QWIIC, J48 JP_VIN, J49 JP_5V, J5 SERVO, J50 JP_3V3, J6 SERVO, J7 SERVO, J8 LED_OUT, J9 LED_OUT, K1 HK4100F-DC5V-SHG, K2 HK4100F-DC5V-SHG, K3 HK4100F-DC5V-SHG, Q1 AO3400A, Q2 AO3400A, Q3 AO3400A, Q4 AO3400A, Q5 AO3400A, Q6 AO3400A, Q7 AOD4185, Q8 AO3400A, SW1 TS-1187A, SW2 TS-1187A, U1 USBLC6-2SC6, U10 PCM5102APWR, U11 SN74AHCT541, U2 ESP32-S3-WROOM-1U-N8R2, U3 ULN2003A, U4 PCA9685PW, U5 AP64350SP-13, U6 TLV62569DBV, U7 DRV8871DDAR, U8 DRV8871DDAR, U9 MAX98357AETE+T

Commit message: Pro v0.1: board setup + placement, two design reviews applied, datasheet-review changes specced
Checkpoint of two weeks' work since dacce25. The schematic is MID-EDIT:
sheets 02/04/05/07/08 checkers are red by design until the changes in
hardware/pro/schematic-changes-2026-09-16.md are drawn; sheet 03 is
half-drawn (see finish-v0.1.md).

Layout
- layout.md rebuilt as one ordered procedure (Part A) with a
  where-you-are line; Board Setup, outline, origin, frozen 120x90 hole
  pattern; routing and pour guidance; per-net noise keep-outs
- tools: checksetup.py (setup/outline/holes/netclasses/socket rows),
  placeboard.py, placetps.py (test points on B.Cu for bodge + pogo rig),
  setpos.py, snapgrid.py; placement renders; power/MCU placement tables

Reviews
- review-2026-09-08 (external audit): C1 EN cap, MA/MB_ILIM short,
  servo/output channel order, sensor clamp order, VIN_FUSED label,
  F1 footprint — all fixed in the schematic
- checknet.py: merged-net assertion (distinct spec nets must be
  distinct schematic nets) — the class that hid the ILIM short
- review-2026-09-16 (routing) + datasheet-review-2026-09-16 with a
  verified disposition; Mini plan audit + recommendations (other session)

Decisions 2026-09-16 (specs, pinmap and headers updated; drawing pending)
- 5 V rail: strip bulk 1000 uF -> 220 uF Rubycon C88757; JP_USB link
  makes USB power opt-in (AP64350 hiccups into 2 mF)
- sensor series R 1 k 0603 -> 2.2 k 1206 C17948 (24 V miswire)
- second PCA9685 (0x41, 1 kHz) for the six DC channels; servos stay at
  50 Hz on 0x40; both OE on GPIO 37 = PCA_OE with pull-up (pinmap:
  36/36 GPIO used; genpins.py supports several PCA9685s)
- output FETs Q1-Q6 -> 40 V Vishay SI2356DS C74127 (TVS coordination)
- SD DAT1/DAT2 pull-ups; USB 22R pair + DNP caps + VBUS 100 nF;
  74AHCT541 input pulldowns, R53 fitted
- MP6603 dual-mode socket mapping verified; MS strap defaults decided

Co-Authored-By: Claude Opus 5 (1M context) <noreply@anthropic.com>
Parts:
- added REF**: MountingHole_3.2mm_M3, MountingHole:MountingHole_3.2mm_M3, F.Cu at (74.8, 51.2)
- added REF**: MountingHole_3.2mm_M3, MountingHole:MountingHole_3.2mm_M3, F.Cu at (194.8, 141.2)
- added REF**: MountingHole_3.2mm_M3, MountingHole:MountingHole_3.2mm_M3, F.Cu at (74.8, 141.2)
- added REF**: MountingHole_3.2mm_M3, MountingHole:MountingHole_3.2mm_M3, F.Cu at (194.8, 51.2)
- TP1, TP10, TP11, TP12, TP13, TP14, TP15, TP16, TP17, TP18, TP19, TP2, TP20, TP21, TP22, TP23, TP24, TP25, TP26, TP27, TP28, TP29, TP3, TP30, TP31, TP32, TP33, TP34, TP35, TP36, TP37, TP38, TP39, TP4, TP40, TP41, TP5, TP6, TP7, TP8, TP9: moved to B.Cu
- moved R38 523.7 mm to (118.0, 103.8), turned to -90 degrees
- moved R37 521.9 mm to (120.0, 103.8), turned to -90 degrees
- moved R36 519.8 mm to (122.0, 103.8), turned to -90 degrees
- moved C43 518.4 mm to (115.5, 129.2)
- moved R34 518.0 mm to (124.0, 103.8), turned to -90 degrees
- moved R35 516.2 mm to (126.0, 103.8), turned to -90 degrees
- moved C42 515.3 mm to (127.0, 101.2), turned to 180 degrees
- moved U11 512.1 mm to (122.0, 94.0), turned to -90 degrees
- moved J38 512.0 mm to (114.2, 140.8)
- moved C45 504.2 mm to (128.8, 129.2)
- moved C44 503.7 mm to (138.2, 96.2), turned to -90 degrees
- moved J37 500.8 mm to (124.2, 140.8)
- moved LED1 496.0 mm to (134.8, 96.2)
- moved J39 489.7 mm to (134.2, 140.8)
- moved J36 478.8 mm to (144.2, 140.8)
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- renumbered J9 to J10, J7 to J6, J6 to J7, J10 to J9
Connections:
- net Net-(J48-Pin_2) renamed /Power/VIN_BUCK
- net Net-(J49-Pin_2) renamed /Power/5V_BUCK
- net Net-(J50-Pin_2) renamed /Power/3V3_BUCK
- net Net-(Q7-D) renamed /Power/VIN_FUSED
- D12 pad 3: /Sensor Expansion/DI1_RAW -> DIGITAL_IN_1
- D13 pad 3: /Sensor Expansion/DI2_RAW -> DIGITAL_IN_2
- D14 pad 3: /Sensor Expansion/DI3_RAW -> DIGITAL_IN_3
- R24 pad 1: /Motors/MA_ILIM -> /Motors/MB_ILIM
- U8 pad 4: /Motors/MA_ILIM -> /Motors/MB_ILIM
Other:
- outline, holes or cut-outs redrawn
- copper layers 2 -> 4

Commit message: Pro v0.1 schematic complete; board cleanup pass, parity 0
Schematic: all datasheet-review changes drawn (decisions 1A, 2A, 3B,
OE on GPIO 37, 4B). All eight sheet checkers ALL NETS MATCH, ERC 0
errors / 0 warnings, pinmap matches generated headers.
- sheet 03: second PCA9685 (U12, 0x41) with B-straps, PCA_OE net with
  10k pull-up (R59); DC FETs Q1-Q6 = SI2356DS
- sheets 02/04/05/07/08: USB link/22R/VBUS cap, SD DAT1/DAT2 pull-ups,
  shifter pulldowns, 2.2k 1206 sensor Rs; R53 (GPIO3 pulldown) now drawn
  on sheet 05, specs moved to match

Board (KiCad closed, backup kept):
- F8 done, schematic parity 0; orphan DNP R53 removed
- mounting holes H1-H4, board-only, excluded from BOM/position files
- minimum drill 0.3 -> 0.2 mm: U2's own 0.2/0.6 thermal vias; JLCPCB
  4-layer standard cost for 0.2 mm holes with >= 0.45 mm pads
- DG128-02P pads 2.3 -> 2.8 mm (J17 10 A input; library edited too)
- DRV8871 exposed-pad paste inset 0.1 mm (library edited too)
- 43 parts snapped to grid; snapgrid.py now exempts J20/J22 so the
  StepStick rows stay 12.70 mm
- DRC: 11 courtyard overlaps left (3 accepted terminal gangs, 8 in the
  sensor corner from the 1206 resistors) + silkscreen

Tools: checknet.py net vote ignores orientation for R/C/L (three
upside-down pull-ups had out-voted the chip pin on sheet 04); verified
it still catches a shorted net and a mis-wired pull-up.
checksetup.py: min drill 0.2.

Also includes the Mini module selection and KiCad project started in
another session (2026-09-19).

Co-Authored-By: Claude Opus 5.5 <noreply@anthropic.com>
Parts:
- added C48: 10U, Capacitor_SMD:C_0805_2012Metric, F.Cu at (119.0, 68.5)
- added C49: 100n, Capacitor_SMD:C_0603_1608Metric, F.Cu at (121.0, 68.5)
- added C50: 100n, Capacitor_SMD:C_0603_1608Metric, F.Cu at (115.2, 58.2)
- added C51: DNP, Capacitor_SMD:C_0603_1608Metric, F.Cu at (106.5, 64.5)
- added C52: DNP, Capacitor_SMD:C_0603_1608Metric, F.Cu at (106.5, 62.8)
- added J51: JP_USB, Connector_PinHeader_2.54mm:PinHeader_1x02_P2.54mm_Vertical, F.Cu at (112.2, 67.8)
- added R54: 10k, Resistor_SMD:R_0603_1608Metric, F.Cu at (109.0, 71.8)
- added R55: 10k, Resistor_SMD:R_0603_1608Metric, F.Cu at (109.0, 73.5)
- added R56: 10k, Resistor_SMD:R_0603_1608Metric, F.Cu at (109.0, 75.2)
- added R57: 10k, Resistor_SMD:R_0603_1608Metric, F.Cu at (109.0, 77.0)
- added R58: 10k, Resistor_SMD:R_0603_1608Metric, F.Cu at (109.0, 78.8)
- added R59: 10k, Resistor_SMD:R_0603_1608Metric, F.Cu at (120.8, 72.0)
- added R60: 10k, Resistor_SMD:R_0603_1608Metric, F.Cu at (122.2, 72.0)
- added R61: 10K, Resistor_SMD:R_0603_1608Metric, F.Cu at (125.5, 85.8)
- added R62: 10K, Resistor_SMD:R_0603_1608Metric, F.Cu at (122.2, 85.8)
- added R63: 10K, Resistor_SMD:R_0603_1608Metric, F.Cu at (120.8, 85.8)
- added R64: 10K, Resistor_SMD:R_0603_1608Metric, F.Cu at (119.2, 85.8)
- added R65: 10K, Resistor_SMD:R_0603_1608Metric, F.Cu at (133.2, 64.5)
- added R66: 10K, Resistor_SMD:R_0603_1608Metric, F.Cu at (121.5, 64.5)
- added R67: 22R, Resistor_SMD:R_0603_1608Metric, F.Cu at (109.8, 64.5)
- added R68: 22R, Resistor_SMD:R_0603_1608Metric, F.Cu at (109.8, 62.8)
- added U12: PCA9685PW, Package_SO:TSSOP-28_4.4x9.7mm_P0.65mm, F.Cu at (115.2, 75.8)
- C43, C45: value 1000u/16V -> 220u/16V; footprint Capacitor_THT:CP_Radial_D10.0mm_P5.00mm -> Capacitor_THT:CP_Radial_D6.3mm_P2.50mm
- Q1, Q2, Q3, Q4, Q5, Q6: value AO3400A -> SI2356DS
- R40, R47, R52: value 1k -> 2.2k; footprint Resistor_SMD:R_0603_1608Metric -> Resistor_SMD:R_1206_3216Metric
- R53: value DNP -> 10k
- TP1: value TP37 -> PCA_OE
- moved C5 19.4 mm to (133.2, 68.8), turned to 90 degrees
- moved C4 18.4 mm to (131.2, 68.8), turned to 90 degrees
- moved R5 15.0 mm to (133.2, 72.0)
- moved R53 14.3 mm to (124.0, 85.8)
- moved R7 12.6 mm to (121.5, 74.8), turned to 180 degrees
- moved R6 12.6 mm to (133.2, 75.2)
- moved R8 9.84 mm to (121.5, 76.2), turned to 180 degrees
- moved R12 8.36 mm to (133.2, 78.5)
- moved R9 7.46 mm to (121.5, 77.8), turned to 180 degrees
- moved U4 7.16 mm to (128.2, 75.8), turned to 0 degrees
- moved R10 5.59 mm to (121.5, 79.5), turned to 180 degrees
- moved R11 5.48 mm to (121.5, 81.0), turned to 180 degrees
- moved D1 3.34 mm to (115.2, 63.0)
- moved J36 0.14 mm to (144.2, 140.8)
- moved J37 0.14 mm to (124.2, 140.8)
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- renumbered REF** to H1, REF** to H2, REF** to H3, REF** to H4
Connections:
- Card1 pad 1: unconnected-(Card1-DAT2(RSV)-Pad1) -> Net-(Card1-DAT2(RSV))
- Card1 pad 8: unconnected-(Card1-DAT1(RSV)-Pad8) -> Net-(Card1-DAT1(RSV))
- D1 pad 1: +5V -> Net-(D1-K)
- J1 pad A6: USB_DP -> USB_DP_CONN
- J1 pad A7: USB_DM -> USB_DM_CONN
- J1 pad B6: USB_DP -> USB_DP_CONN
- J1 pad B7: USB_DM -> USB_DM_CONN
- TP1 pad 1: Net-(U2-IO37) -> PCA_OE
- U1 pad 1: USB_DM -> USB_DM_CONN
- U1 pad 3: USB_DP -> USB_DP_CONN
- U1 pad 4: USB_DP -> USB_DP_CONN
- U1 pad 6: USB_DM -> USB_DM_CONN
- U2 pad 30: Net-(U2-IO37) -> PCA_OE
- U4 pad 12: /Outputs/LED_1 -> unconnected-(U4-LED6-Pad12)
- U4 pad 13: /Outputs/LED_2 -> unconnected-(U4-LED7-Pad13)
- U4 pad 15: /Outputs/LED_3 -> unconnected-(U4-LED8-Pad15)
- U4 pad 16: /Outputs/LED_4 -> unconnected-(U4-LED9-Pad16)
- U4 pad 17: /Outputs/LED_5 -> unconnected-(U4-LED10-Pad17)
- U4 pad 18: /Outputs/LED_6 -> unconnected-(U4-LED11-Pad18)
- U4 pad 23: GND -> PCA_OE
