File: hardware/pro/propmesh/testpoints.kicad_sch (KiCad schematic)
At the start: 40 parts

Commit message: Pro v0.1 schematic complete; board cleanup pass, parity 0
Schematic: all datasheet-review changes drawn (decisions 1A, 2A, 3B,
OE on GPIO 37, 4B). All eight sheet checkers ALL NETS MATCH, ERC 0
errors / 0 warnings, pinmap matches generated headers.
- sheet 03: second PCA9685 (U12, 0x41) with B-straps, PCA_OE net with
  10k pull-up (R59); DC FETs Q1-Q6 = SI2356DS
- sheets 02/04/05/07/08: USB link/22R/VBUS cap, SD DAT1/DAT2 pull-ups,
  shifter pulldowns, 2.2k 1206 sensor Rs; R53 (GPIO3 pulldown) now drawn
  on sheet 05, specs moved to match

Board (KiCad closed, backup kept):
- F8 done, schematic parity 0; orphan DNP R53 removed
- mounting holes H1-H4, board-only, excluded from BOM/position files
- minimum drill 0.3 -> 0.2 mm: U2's own 0.2/0.6 thermal vias; JLCPCB
  4-layer standard cost for 0.2 mm holes with >= 0.45 mm pads
- DG128-02P pads 2.3 -> 2.8 mm (J17 10 A input; library edited too)
- DRV8871 exposed-pad paste inset 0.1 mm (library edited too)
- 43 parts snapped to grid; snapgrid.py now exempts J20/J22 so the
  StepStick rows stay 12.70 mm
- DRC: 11 courtyard overlaps left (3 accepted terminal gangs, 8 in the
  sensor corner from the 1206 resistors) + silkscreen

Tools: checknet.py net vote ignores orientation for R/C/L (three
upside-down pull-ups had out-voted the chip pin on sheet 04); verified
it still catches a shorted net and a mis-wired pull-up.
checksetup.py: min drill 0.2.

Also includes the Mini module selection and KiCad project started in
another session (2026-09-19).

Co-Authored-By: Claude Opus 5.5 <noreply@anthropic.com>
Parts:
- removed R53: DNP, Resistor_SMD:R_0603_1608Metric, symbol Device:R
Changed lines of the file:
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@@
 	(wire
 		(pts
-			(xy 236.22 111.76) (xy 241.3 111.76)
-		)
-		(stroke
-			(width 0)
-			(type default)
-		)
-	)
-	(wire
-		(pts
 			(xy 236.22 74.93) (xy 241.3 74.93)
 		)
@@
 		)
 	)
-	(global_label "LED_STRIP_1_CLK"
-		(shape input)
-		(at 241.3 111.76 0)
-		(fields_autoplaced yes)
-		(effects
-			(font
-				(size 1.27 1.27)
-			)
-			(justify left)
-		)
-		(property "Intersheetrefs" "${INTERSHEET_REFS}"
-			(at 241.8 111.76 0)
-			(hide yes)
-			(show_name no)
-			(do_not_autoplace no)
-			(effects
-				(font
-					(size 1.27 1.27)
-				)
-				(justify left)
-			)
-		)
-	)
 	(global_label "VIN_RAW"
 		(shape input)
@@
 	)
 	(symbol
-		(lib_id "Device:R")
-		(at 236.22 115.57 0)
-		(unit 1)
-		(body_style 1)
-		(exclude_from_sim no)
-		(in_bom yes)
-		(on_board yes)
-		(in_pos_files yes)
-		(dnp yes)
-		(fields_autoplaced yes)
-		(property "Reference" "R53"
-			(at 238.76 114.3 0)
-			(show_name no)
-			(do_not_autoplace no)
-			(effects
-				(font
-					(size 1.27 1.27)
-				)
-				(justify left)
-			)
-		)
-		(property "Value" "DNP"
-			(at 238.76 116.84 0)
-			(show_name no)
-			(do_not_autoplace no)
-			(effects
-				(font
-					(size 1.27 1.27)
-				)
-				(justify left)
-			)
-		)
-		(property "Footprint" "Resistor_SMD:R_0603_1608Metric"
-			(at 234.442 115.57 90)
-			(hide yes)
-			(show_name no)
-			(do_not_autoplace no)
-			(effects
-				(font
-					(size 1.27 1.27)
-				)
-			)
-		)
-		(property "Datasheet" ""
-			(at 236.22 115.57 0)
-			(hide yes)
-			(show_name no)
-			(do_not_autoplace no)
-			(effects
-				(font
-					(size 1.27 1.27)
-				)
-			)
-		)
-		(property "Description" "Resistor"
-			(at 236.22 115.57 0)
-			(hide yes)
-			(show_name no)
-			(do_not_autoplace no)
-			(effects
-				(font
-					(size 1.27 1.27)
-				)
-			)
-		)
-		(pin "2"
-		)
-		(pin "1"
-		)
-		(instances
-			(project "propmesh"
-				(path "/6aa579d1-bfe0-499b-882d-72f52ff6d36c/3e4ac41d-339a-48df-ae9d-b064c7089ccd"
-					(reference "R53")
-					(unit 1)
-				)
-			)
-		)
-	)
-	(symbol
 		(lib_id "Connector:TestPoint")
 		(at 29.21 39.37 0)
@@
 					(unit 1)
 				)
-			)
-		)
-	)
-	(symbol
-		(lib_id "power:GND")
-		(at 236.22 119.38 0)
-		(unit 1)
-		(body_style 1)
-		(exclude_from_sim no)
-		(in_bom yes)
-		(on_board yes)
-		(in_pos_files yes)
-		(dnp no)
-		(fields_autoplaced yes)
-		(property "Reference" "#PWR0195"
-			(at 236.22 125.73 0)
-			(hide yes)
-			(show_name no)
-			(do_not_autoplace no)
-			(effects
-				(font
-					(size 1.27 1.27)
-				)
-			)
-		)
-		(property "Value" "GND"
-			(at 236.22 124.46 0)
-			(show_name no)
-			(do_not_autoplace no)
-			(effects
-				(font
-					(size 1.27 1.27)
-				)
-			)
-		)
-		(property "Footprint" ""
-			(at 236.22 119.38 0)
-			(hide yes)
-			(show_name no)
-			(do_not_autoplace no)
-			(effects
-				(font
-					(size 1.27 1.27)
-				)
-			)
-		)
-		(property "Datasheet" ""
-			(at 236.22 119.38 0)
-			(hide yes)
-			(show_name no)
-			(do_not_autoplace no)
-			(effects
-				(font
-					(size 1.27 1.27)
-				)
-			)
-		)
-		(property "Description" "Power symbol creates a global label with name \"GND\" , ground"
-			(at 236.22 119.38 0)
-			(hide yes)
-			(show_name no)
-			(do_not_autoplace no)
-			(effects
-				(font
-					(size 1.27 1.27)
-				)
-			)
-		)
-		(pin "1"
-		)
-		(instances
-			(project "propmesh"
-				(path "/6aa579d1-bfe0-499b-882d-72f52ff6d36c/3e4ac41d-339a-48df-ae9d-b064c7089ccd"
-					(reference "#PWR0195")
-					(unit 1)
-				)
